File: 0_Castor/keyswitches.kicad_sch (KiCad schematic)
At the start: 84 parts

Commit message: feat: add controller, battery jack, battery switch and reset switch placement
Parts:
- S48: footprint ScottoKeebs_Hotswap:Hotswap_MX_1.00u -> ScottoKeebs_Hotswap:Hotswap_MX_2.00u
Changed lines of the file:
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@@
 			)
 		)
-		(property "Footprint" "ScottoKeebs_Hotswap:Hotswap_MX_1.00u"
+		(property "Footprint" "ScottoKeebs_Hotswap:Hotswap_MX_2.00u"
 			(at 59.69 120.65 0)
 			(hide yes)
