File: 0_Castor/leds.kicad_sch (KiCad schematic)
At the start: 44 parts

Commit message: feat: add controller, battery jack, battery switch and reset switch placement
Parts:
- added R1, R2, R3, R4: Resistor, ScottoKeebs_Components:Resistor_0402, symbol ScottoKeebs:Placeholder_Resistor
Connections:
- net at LED44.1 (DOUT): now also R4.1
- net at LED25.1 (DOUT): now also R3.1
- net DIN 0: no longer names the net of LED1.3 (DIN)
- net DIN 0: now also R2.2
- net DIN 1: no longer names the net of LED26.3 (DIN)
- net DIN 1: now also R1.2
- new net DIN0: R2.1
- new net DIN1: R1.1
- new net DOUT0: R3.2
- new net DOUT1: R4.2
