File: 0_Castor/_leds.kicad_sch (KiCad schematic)
At the start: 90 parts

Commit message: feat: convert 3.3V from nice!nano to 5V to LEDs
Parts:
- C1, C10, C11, C12, C13, C14, C15, C16, C17, C18, C19, C2, C20, C21, C22, C23, C24, C25, C26, C27, C28, C29, C3, C30, C31, C32, C33, C34, C35, C36, C37, C38, C39, C4, C40, C41, C42, C43, C44, C5, C6, C7, C8, C9: footprint Capacitor_SMD:C_0402_1005Metric -> Capacitor_SMD:C_0603_1608Metric
- R1, R2: footprint Resistor_SMD:R_0402_1005Metric -> Resistor_SMD:R_0603_1608Metric
Connections:
- net DIN renamed Voltage booster/D_{5V}
- net DOUT renamed D_{OUT}
- net VDD renamed +5V_{LED}
Other:
- added sheet Voltage booster (_voltage_booster.kicad_sch)

Commit message: feat: add voltage booster for LEDs power supply
Parts:
- added R5: 200Ω, Resistor_SMD:R_0603_1608Metric, symbol Device:R_Small_US
Connections:
- net +5V_{LED}: now also R5.1
- net D_{OUT} renamed LED_{OUT}
- net Voltage booster/D_{5V} renamed Voltage booster/5V_{INPUT}
- new net +5V: R5.2
Other:
- sheet Voltage booster ports: added 3.3V_{INPUT}, 5V_{INPUT}; removed D_{3.3V}, D_{5V}
