File: 0_Castor/_keyswitches.kicad_sch (KiCad schematic)
At the start: 84 parts

Commit message: feat: add LEDs, capacitors, resistors and rework schematic
Parts:
- renumbered D45 to D1, D58 to D10, D64 to D11, D71 to D12, D79 to D13, D46 to D14, D53 to D15, D59 to D16, D65 to D17, D72 to D18, D80 to D19, D51 to D2, D47 to D20, D54 to D21, D60 to D22, D66 to D23, D73 to D24, D81 to D25, D48 to D26, D55 to D27, D61 to D28, D67 to D29, D57 to D3, D74 to D30, D82 to D31, D44 to D32, D50 to D33, D56 to D34, D62 to D35, D75 to D36, D68 to D37, D76 to D38, D83 to D39, D63 to D4, D69 to D40, D77 to D41, D84 to D42, D70 to D5, D78 to D6, D43 to D7, D49 to D8, D52 to D9, S45 to S1, S58 to S10, S64 to S11, S71 to S12, S79 to S13, S46 to S14, S53 to S15, S59 to S16, S65 to S17, S72 to S18, S80 to S19, S51 to S2, S47 to S20, S54 to S21, S60 to S22, S66 to S23, S73 to S24, S81 to S25, S48 to S26, S55 to S27, S61 to S28, S67 to S29, S57 to S3, S74 to S30, S82 to S31, S44 to S32, S50 to S33, S56 to S34, S62 to S35, S75 to S36, S68 to S37, S76 to S38, S83 to S39, S63 to S4, S69 to S40, S77 to S41, S84 to S42, S70 to S5, S78 to S6, S43 to S7, S49 to S8, S52 to S9
Other:
- moved on the sheet: D1, D10, D11, D12, D13, D14, D15, D16, D17, D18, D19, D2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

Commit message: feat: remove LED's and place components in PCB
Parts:
- S1, S14, S20, S26: footprint ScottoKeebs_Hotswap:Hotswap_MX_2.00u -> ScottoKeebs_Hotswap:Hotswap_Choc_V2_2.00u
- S10, S11, S12, S13, S15, S16, S17, S18, S19, S2, S21, S22, S23, S24, S25, S27, S28, S29, S3, S30, S31, S32, S33, S34, S35, S37, S38, S39, S4, S40, S41, S42, S5, S6, S7, S8, S9: footprint ScottoKeebs_Hotswap:Hotswap_MX_1.00u -> ScottoKeebs_Hotswap:Hotswap_Choc_V2_1.00u
- S36: footprint ScottoKeebs_Hotswap:Hotswap_MX_3.00u -> ScottoKeebs_Hotswap:Hotswap_Choc_V2_3.00u
Changed lines of the file:
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@@
 			)
 		)
-		(property "Footprint" "ScottoKeebs_Hotswap:Hotswap_MX_1.00u"
+		(property "Footprint" "ScottoKeebs_Hotswap:Hotswap_Choc_V2_1.00u"
 			(at 67.31 102.87 0)
 			(hide yes)
@@
 			)
 		)
-		(property "Footprint" "ScottoKeebs_Hotswap:Hotswap_MX_1.00u"
+		(property "Footprint" "ScottoKeebs_Hotswap:Hotswap_Choc_V2_1.00u"
 			(at 80.01 53.34 0)
 			(hide yes)
@@
 			)
 		)
-		(property "Footprint" "ScottoKeebs_Hotswap:Hotswap_MX_1.00u"
+		(property "Footprint" "ScottoKeebs_Hotswap:Hotswap_Choc_V2_1.00u"
 			(at 80.01 152.4 0)
 			(hide yes)
@@
 			)
 		)
-		(property "Footprint" "ScottoKeebs_Hotswap:Hotswap_MX_1.00u"
+		(property "Footprint" "ScottoKeebs_Hotswap:Hotswap_Choc_V2_1.00u"
 			(at 54.61 86.36 0)
 			(hide yes)
@@
 			)
 		)
-		(property "Footprint" "ScottoKeebs_Hotswap:Hotswap_MX_1.00u"
+		(property "Footprint" "ScottoKeebs_Hotswap:Hotswap_Choc_V2_1.00u"
 			(at 105.41 36.83 0)
 			(hide yes)
@@
 			)
 		)
-		(property "Footprint" "ScottoKeebs_Hotswap:Hotswap_MX_1.00u"
+		(property "Footprint" "ScottoKeebs_Hotswap:Hotswap_Choc_V2_1.00u"
 			(at 92.71 135.89 0)
 			(hide yes)
@@
 			)
 		)
-		(property "Footprint" "ScottoKeebs_Hotswap:Hotswap_MX_1.00u"
+		(property "Footprint" "ScottoKeebs_Hotswap:Hotswap_Choc_V2_1.00u"
 			(at 54.61 36.83 0)
 			(hide yes)
@@
 			)
 		)
-		(property "Footprint" "ScottoKeebs_Hotswap:Hotswap_MX_1.00u"
+		(property "Footprint" "ScottoKeebs_Hotswap:Hotswap_Choc_V2_1.00u"
 			(at 80.01 69.85 0)
 			(hide yes)
@@
 			)
 		)
-		(property "Footprint" "ScottoKeebs_Hotswap:Hotswap_MX_1.00u"
+		(property "Footprint" "ScottoKeebs_Hotswap:Hotswap_Choc_V2_1.00u"
 			(at 92.71 102.87 0)
 			(hide yes)
@@
 			)
 		)
-		(property "Footprint" "ScottoKeebs_Hotswap:Hotswap_MX_1.00u"
+		(property "Footprint" "ScottoKeebs_Hotswap:Hotswap_Choc_V2_1.00u"
 			(at 29.21 119.38 0)
 			(hide yes)
@@
 			)
 		)
-		(property "Footprint" "ScottoKeebs_Hotswap:Hotswap_MX_1.00u"
+		(property "Footprint" "ScottoKeebs_Hotswap:Hotswap_Choc_V2_1.00u"
 			(at 67.31 86.36 0)
 			(hide yes)
@@
 			)
 		)
-		(property "Footprint" "ScottoKeebs_Hotswap:Hotswap_MX_1.00u"
+		(property "Footprint" "ScottoKeebs_Hotswap:Hotswap_Choc_V2_1.00u"
 			(at 80.01 102.87 0)
 			(hide yes)
@@
 			)
 		)
-		(property "Footprint" "ScottoKeebs_Hotswap:Hotswap_MX_1.00u"
+		(property "Footprint" "ScottoKeebs_Hotswap:Hotswap_Choc_V2_1.00u"
 			(at 105.41 86.36 0)
 			(hide yes)
@@
 			)
 		)
-		(property "Footprint" "ScottoKeebs_Hotswap:Hotswap_MX_1.00u"
+		(property "Footprint" "ScottoKeebs_Hotswap:Hotswap_Choc_V2_1.00u"
 			(at 80.01 86.36 0)
 			(hide yes)
@@
 			)
 		)
-		(property "Footprint" "ScottoKeebs_Hotswap:Hotswap_MX_1.00u"
+		(property "Footprint" "ScottoKeebs_Hotswap:Hotswap_Choc_V2_1.00u"
 			(at 105.41 135.89 0)
 			(hide yes)
@@
 			)
 		)
-		(property "Footprint" "ScottoKeebs_Hotswap:Hotswap_MX_1.00u"
+		(property "Footprint" "ScottoKeebs_Hotswap:Hotswap_Choc_V2_1.00u"
 			(at 105.41 152.4 0)
 			(hide yes)
@@
 			)
 		)
-		(property "Footprint" "ScottoKeebs_Hotswap:Hotswap_MX_2.00u"
+		(property "Footprint" "ScottoKeebs_Hotswap:Hotswap_Choc_V2_2.00u"
 			(at 35.56 86.36 0)
 			(hide yes)
@@
 			)
 		)
-		(property "Footprint" "ScottoKeebs_Hotswap:Hotswap_MX_3.00u"
+		(property "Footprint" "ScottoKeebs_Hotswap:Hotswap_Choc_V2_3.00u"
 			(at 92.71 119.38 0)
 			(hide yes)
@@
 			)
 		)
-		(property "Footprint" "ScottoKeebs_Hotswap:Hotswap_MX_1.00u"
+		(property "Footprint" "ScottoKeebs_Hotswap:Hotswap_Choc_V2_1.00u"
 			(at 54.61 53.34 0)
 			(hide yes)
@@
 			)
 		)
-		(property "Footprint" "ScottoKeebs_Hotswap:Hotswap_MX_2.00u"
+		(property "Footprint" "ScottoKeebs_Hotswap:Hotswap_Choc_V2_2.00u"
 			(at 35.56 36.83 0)
 			(hide yes)
@@
 			)
 		)
-		(property "Footprint" "ScottoKeebs_Hotswap:Hotswap_MX_1.00u"
+		(property "Footprint" "ScottoKeebs_Hotswap:Hotswap_Choc_V2_1.00u"
 			(at 41.91 119.38 0)
 			(hide yes)
@@
 			)
 		)
-		(property "Footprint" "ScottoKeebs_Hotswap:Hotswap_MX_1.00u"
+		(property "Footprint" "ScottoKeebs_Hotswap:Hotswap_Choc_V2_1.00u"
 			(at 54.61 119.38 0)
 			(hide yes)
@@
 			)
 		)
-		(property "Footprint" "ScottoKeebs_Hotswap:Hotswap_MX_1.00u"
+		(property "Footprint" "ScottoKeebs_Hotswap:Hotswap_Choc_V2_1.00u"
 			(at 92.71 53.34 0)
 			(hide yes)
@@
 			)
 		)
-		(property "Footprint" "ScottoKeebs_Hotswap:Hotswap_MX_1.00u"
+		(property "Footprint" "ScottoKeebs_Hotswap:Hotswap_Choc_V2_1.00u"
 			(at 105.41 69.85 0)
 			(hide yes)
@@
 			)
 		)
-		(property "Footprint" "ScottoKeebs_Hotswap:Hotswap_MX_1.00u"
+		(property "Footprint" "ScottoKeebs_Hotswap:Hotswap_Choc_V2_1.00u"
 			(at 54.61 69.85 0)
 			(hide yes)
@@
 			)
 		)
-		(property "Footprint" "ScottoKeebs_Hotswap:Hotswap_MX_2.00u"
+		(property "Footprint" "ScottoKeebs_Hotswap:Hotswap_Choc_V2_2.00u"
 			(at 35.56 69.85 0)
 			(hide yes)
@@
 			)
 		)
-		(property "Footprint" "ScottoKeebs_Hotswap:Hotswap_MX_2.00u"
+		(property "Footprint" "ScottoKeebs_Hotswap:Hotswap_Choc_V2_2.00u"
 			(at 35.56 102.87 0)
 			(hide yes)
@@
 			)
 		)
-		(property "Footprint" "ScottoKeebs_Hotswap:Hotswap_MX_1.00u"
+		(property "Footprint" "ScottoKeebs_Hotswap:Hotswap_Choc_V2_1.00u"
 			(at 67.31 36.83 0)
 			(hide yes)
@@
 			)
 		)
-		(property "Footprint" "ScottoKeebs_Hotswap:Hotswap_MX_1.00u"
+		(property "Footprint" "ScottoKeebs_Hotswap:Hotswap_Choc_V2_1.00u"
 			(at 105.41 53.34 0)
 			(hide yes)
@@
 			)
 		)
-		(property "Footprint" "ScottoKeebs_Hotswap:Hotswap_MX_1.00u"
+		(property "Footprint" "ScottoKeebs_Hotswap:Hotswap_Choc_V2_1.00u"
 			(at 80.01 36.83 0)
 			(hide yes)
@@
 			)
 		)
-		(property "Footprint" "ScottoKeebs_Hotswap:Hotswap_MX_1.00u"
+		(property "Footprint" "ScottoKeebs_Hotswap:Hotswap_Choc_V2_1.00u"
 			(at 105.41 102.87 0)
 			(hide yes)
@@
 			)
 		)
-		(property "Footprint" "ScottoKeebs_Hotswap:Hotswap_MX_1.00u"
+		(property "Footprint" "ScottoKeebs_Hotswap:Hotswap_Choc_V2_1.00u"
 			(at 41.91 53.34 0)
 			(hide yes)
@@
 			)
 		)
-		(property "Footprint" "ScottoKeebs_Hotswap:Hotswap_MX_1.00u"
+		(property "Footprint" "ScottoKeebs_Hotswap:Hotswap_Choc_V2_1.00u"
 			(at 67.31 119.38 0)
 			(hide yes)
@@
 			)
 		)
-		(property "Footprint" "ScottoKeebs_Hotswap:Hotswap_MX_1.00u"
+		(property "Footprint" "ScottoKeebs_Hotswap:Hotswap_Choc_V2_1.00u"
 			(at 67.31 69.85 0)
 			(hide yes)
@@
 			)
 		)
-		(property "Footprint" "ScottoKeebs_Hotswap:Hotswap_MX_1.00u"
+		(property "Footprint" "ScottoKeebs_Hotswap:Hotswap_Choc_V2_1.00u"
 			(at 92.71 69.85 0)
 			(hide yes)
@@
 			)
 		)
-		(property "Footprint" "ScottoKeebs_Hotswap:Hotswap_MX_1.00u"
+		(property "Footprint" "ScottoKeebs_Hotswap:Hotswap_Choc_V2_1.00u"
 			(at 92.71 36.83 0)
 			(hide yes)
@@
 			)
 		)
-		(property "Footprint" "ScottoKeebs_Hotswap:Hotswap_MX_1.00u"
+		(property "Footprint" "ScottoKeebs_Hotswap:Hotswap_Choc_V2_1.00u"
 			(at 80.01 135.89 0)
 			(hide yes)
@@
 			)
 		)
-		(property "Footprint" "ScottoKeebs_Hotswap:Hotswap_MX_1.00u"
+		(property "Footprint" "ScottoKeebs_Hotswap:Hotswap_Choc_V2_1.00u"
 			(at 54.61 102.87 0)
 			(hide yes)
@@
 			)
 		)
-		(property "Footprint" "ScottoKeebs_Hotswap:Hotswap_MX_1.00u"
+		(property "Footprint" "ScottoKeebs_Hotswap:Hotswap_Choc_V2_1.00u"
 			(at 67.31 53.34 0)
 			(hide yes)
@@
 			)
 		)
-		(property "Footprint" "ScottoKeebs_Hotswap:Hotswap_MX_1.00u"
+		(property "Footprint" "ScottoKeebs_Hotswap:Hotswap_Choc_V2_1.00u"
 			(at 92.71 152.4 0)
 			(hide yes)
@@
 			)
 		)
-		(property "Footprint" "ScottoKeebs_Hotswap:Hotswap_MX_1.00u"
+		(property "Footprint" "ScottoKeebs_Hotswap:Hotswap_Choc_V2_1.00u"
 			(at 29.21 53.34 0)
 			(hide yes)
@@
 			)
 		)
-		(property "Footprint" "ScottoKeebs_Hotswap:Hotswap_MX_1.00u"
+		(property "Footprint" "ScottoKeebs_Hotswap:Hotswap_Choc_V2_1.00u"
 			(at 92.71 86.36 0)
 			(hide yes)
