File: 1_Pollux/_keyswitches.kicad_sch (KiCad schematic)
At the start: 98 parts

Commit message: feat: finish Pollux PCB | chore: generate gerber files for both sides
Parts:
- S1, S10, S11, S12, S13, S14, S15, S16, S17, S18, S19, S2, S20, S21, S22, S23, S25, S26, S27, S28, S29, S3, S30, S31, S32, S33, S34, S35, S36, S37, S4, S40, S41, S42, S43, S44, S45, S46, S47, S48, S49, S5, S6, S7, S8, S9: footprint ScottoKeebs_Hotswap:Hotswap_MX_1.00u -> ScottoKeebs_Hotswap:Hotswap_Choc_V2_1.00u
- S24: footprint ScottoKeebs_Hotswap:Hotswap_MX_1.00u -> ScottoKeebs_Hotswap:Hotswap_Choc_V2_2.00u_90deg
- S38: footprint ScottoKeebs_Hotswap:Hotswap_MX_2.00u -> ScottoKeebs_Hotswap:Hotswap_Choc_V2_2.00u
- S39: footprint ScottoKeebs_Hotswap:Hotswap_MX_3.00u -> ScottoKeebs_Hotswap:Hotswap_Choc_V2_3.00u
Changed lines of the file:
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@@
 			)
 		)
-		(property "Footprint" "ScottoKeebs_Hotswap:Hotswap_MX_1.00u"
+		(property "Footprint" "ScottoKeebs_Hotswap:Hotswap_Choc_V2_1.00u"
 			(at 104.14 40.64 0)
 			(hide yes)
@@
 			)
 		)
-		(property "Footprint" "ScottoKeebs_Hotswap:Hotswap_MX_1.00u"
+		(property "Footprint" "ScottoKeebs_Hotswap:Hotswap_Choc_V2_1.00u"
 			(at 78.74 78.74 0)
 			(hide yes)
@@
 			)
 		)
-		(property "Footprint" "ScottoKeebs_Hotswap:Hotswap_MX_1.00u"
+		(property "Footprint" "ScottoKeebs_Hotswap:Hotswap_Choc_V2_1.00u"
 			(at 116.84 40.64 0)
 			(hide yes)
@@
 			)
 		)
-		(property "Footprint" "ScottoKeebs_Hotswap:Hotswap_MX_1.00u"
+		(property "Footprint" "ScottoKeebs_Hotswap:Hotswap_Choc_V2_1.00u"
 			(at 116.84 97.79 0)
 			(hide yes)
@@
 			)
 		)
-		(property "Footprint" "ScottoKeebs_Hotswap:Hotswap_MX_1.00u"
+		(property "Footprint" "ScottoKeebs_Hotswap:Hotswap_Choc_V2_1.00u"
 			(at 53.34 97.79 0)
 			(hide yes)
@@
 			)
 		)
-		(property "Footprint" "ScottoKeebs_Hotswap:Hotswap_MX_1.00u"
+		(property "Footprint" "ScottoKeebs_Hotswap:Hotswap_Choc_V2_1.00u"
 			(at 104.14 97.79 0)
 			(hide yes)
@@
 			)
 		)
-		(property "Footprint" "ScottoKeebs_Hotswap:Hotswap_MX_1.00u"
+		(property "Footprint" "ScottoKeebs_Hotswap:Hotswap_Choc_V2_1.00u"
 			(at 53.34 173.99 0)
 			(hide yes)
@@
 			)
 		)
-		(property "Footprint" "ScottoKeebs_Hotswap:Hotswap_MX_1.00u"
+		(property "Footprint" "ScottoKeebs_Hotswap:Hotswap_Choc_V2_1.00u"
 			(at 40.64 59.69 0)
 			(hide yes)
@@
 			)
 		)
-		(property "Footprint" "ScottoKeebs_Hotswap:Hotswap_MX_1.00u"
+		(property "Footprint" "ScottoKeebs_Hotswap:Hotswap_Choc_V2_1.00u"
 			(at 104.14 78.74 0)
 			(hide yes)
@@
 			)
 		)
-		(property "Footprint" "ScottoKeebs_Hotswap:Hotswap_MX_1.00u"
+		(property "Footprint" "ScottoKeebs_Hotswap:Hotswap_Choc_V2_1.00u"
 			(at 104.14 135.89 0)
 			(hide yes)
@@
 			)
 		)
-		(property "Footprint" "ScottoKeebs_Hotswap:Hotswap_MX_1.00u"
+		(property "Footprint" "ScottoKeebs_Hotswap:Hotswap_Choc_V2_1.00u"
 			(at 91.44 116.84 0)
 			(hide yes)
@@
 			)
 		)
-		(property "Footprint" "ScottoKeebs_Hotswap:Hotswap_MX_1.00u"
+		(property "Footprint" "ScottoKeebs_Hotswap:Hotswap_Choc_V2_1.00u"
 			(at 66.04 154.94 0)
 			(hide yes)
@@
 			)
 		)
-		(property "Footprint" "ScottoKeebs_Hotswap:Hotswap_MX_1.00u"
+		(property "Footprint" "ScottoKeebs_Hotswap:Hotswap_Choc_V2_1.00u"
 			(at 40.64 173.99 0)
 			(hide yes)
@@
 			)
 		)
-		(property "Footprint" "ScottoKeebs_Hotswap:Hotswap_MX_1.00u"
+		(property "Footprint" "ScottoKeebs_Hotswap:Hotswap_Choc_V2_1.00u"
 			(at 78.74 116.84 0)
 			(hide yes)
@@
 			)
 		)
-		(property "Footprint" "ScottoKeebs_Hotswap:Hotswap_MX_1.00u"
+		(property "Footprint" "ScottoKeebs_Hotswap:Hotswap_Choc_V2_1.00u"
 			(at 78.74 97.79 0)
 			(hide yes)
@@
 			)
 		)
-		(property "Footprint" "ScottoKeebs_Hotswap:Hotswap_MX_1.00u"
+		(property "Footprint" "ScottoKeebs_Hotswap:Hotswap_Choc_V2_1.00u"
 			(at 40.64 40.64 0)
 			(hide yes)
@@
 			)
 		)
-		(property "Footprint" "ScottoKeebs_Hotswap:Hotswap_MX_1.00u"
+		(property "Footprint" "ScottoKeebs_Hotswap:Hotswap_Choc_V2_1.00u"
 			(at 91.44 78.74 0)
 			(hide yes)
@@
 			)
 		)
-		(property "Footprint" "ScottoKeebs_Hotswap:Hotswap_MX_1.00u"
+		(property "Footprint" "ScottoKeebs_Hotswap:Hotswap_Choc_V2_1.00u"
 			(at 66.04 173.99 0)
 			(hide yes)
@@
 			)
 		)
-		(property "Footprint" "ScottoKeebs_Hotswap:Hotswap_MX_1.00u"
+		(property "Footprint" "ScottoKeebs_Hotswap:Hotswap_Choc_V2_1.00u"
 			(at 116.84 78.74 0)
 			(hide yes)
@@
 			)
 		)
-		(property "Footprint" "ScottoKeebs_Hotswap:Hotswap_MX_1.00u"
+		(property "Footprint" "ScottoKeebs_Hotswap:Hotswap_Choc_V2_1.00u"
 			(at 104.14 59.69 0)
 			(hide yes)
@@
 			)
 		)
-		(property "Footprint" "ScottoKeebs_Hotswap:Hotswap_MX_1.00u"
+		(property "Footprint" "ScottoKeebs_Hotswap:Hotswap_Choc_V2_1.00u"
 			(at 78.74 59.69 0)
 			(hide yes)
@@
 			)
 		)
-		(property "Footprint" "ScottoKeebs_Hotswap:Hotswap_MX_1.00u"
+		(property "Footprint" "ScottoKeebs_Hotswap:Hotswap_Choc_V2_1.00u"
 			(at 66.04 78.74 0)
 			(hide yes)
@@
 			)
 		)
-		(property "Footprint" "ScottoKeebs_Hotswap:Hotswap_MX_1.00u"
+		(property "Footprint" "ScottoKeebs_Hotswap:Hotswap_Choc_V2_1.00u"
 			(at 40.64 97.79 0)
 			(hide yes)
@@
 			)
 		)
-		(property "Footprint" "ScottoKeebs_Hotswap:Hotswap_MX_1.00u"
+		(property "Footprint" "ScottoKeebs_Hotswap:Hotswap_Choc_V2_1.00u"
 			(at 53.34 116.84 0)
 			(hide yes)
@@
 			)
 		)
-		(property "Footprint" "ScottoKeebs_Hotswap:Hotswap_MX_1.00u"
+		(property "Footprint" "ScottoKeebs_Hotswap:Hotswap_Choc_V2_1.00u"
 			(at 53.34 154.94 0)
 			(hide yes)
@@
 			)
 		)
-		(property "Footprint" "ScottoKeebs_Hotswap:Hotswap_MX_1.00u"
+		(property "Footprint" "ScottoKeebs_Hotswap:Hotswap_Choc_V2_1.00u"
 			(at 40.64 78.74 0)
 			(hide yes)
@@
 			)
 		)
-		(property "Footprint" "ScottoKeebs_Hotswap:Hotswap_MX_2.00u"
+		(property "Footprint" "ScottoKeebs_Hotswap:Hotswap_Choc_V2_2.00u"
 			(at 123.19 116.84 0)
 			(hide yes)
@@
 			)
 		)
-		(property "Footprint" "ScottoKeebs_Hotswap:Hotswap_MX_1.00u"
+		(property "Footprint" "ScottoKeebs_Hotswap:Hotswap_Choc_V2_1.00u"
 			(at 129.54 40.64 0)
 			(hide yes)
@@
 			)
 		)
-		(property "Footprint" "ScottoKeebs_Hotswap:Hotswap_MX_1.00u"
+		(property "Footprint" "ScottoKeebs_Hotswap:Hotswap_Choc_V2_1.00u"
 			(at 40.64 116.84 0)
 			(hide yes)
@@
 			)
 		)
-		(property "Footprint" "ScottoKeebs_Hotswap:Hotswap_MX_1.00u"
+		(property "Footprint" "ScottoKeebs_Hotswap:Hotswap_Choc_V2_1.00u"
 			(at 53.34 40.64 0)
 			(hide yes)
@@
 			)
 		)
-		(property "Footprint" "ScottoKeebs_Hotswap:Hotswap_MX_1.00u"
+		(property "Footprint" "ScottoKeebs_Hotswap:Hotswap_Choc_V2_1.00u"
 			(at 91.44 97.79 0)
 			(hide yes)
@@
 			)
 		)
-		(property "Footprint" "ScottoKeebs_Hotswap:Hotswap_MX_3.00u"
+		(property "Footprint" "ScottoKeebs_Hotswap:Hotswap_Choc_V2_3.00u"
 			(at 53.34 135.89 0)
 			(hide yes)
@@
 			)
 		)
-		(property "Footprint" "ScottoKeebs_Hotswap:Hotswap_MX_1.00u"
+		(property "Footprint" "ScottoKeebs_Hotswap:Hotswap_Choc_V2_1.00u"
 			(at 129.54 59.69 0)
 			(hide yes)
@@
 			)
 		)
-		(property "Footprint" "ScottoKeebs_Hotswap:Hotswap_MX_1.00u"
+		(property "Footprint" "ScottoKeebs_Hotswap:Hotswap_Choc_V2_1.00u"
 			(at 53.34 59.69 0)
 			(hide yes)
@@
 			)
 		)
-		(property "Footprint" "ScottoKeebs_Hotswap:Hotswap_MX_1.00u"
+		(property "Footprint" "ScottoKeebs_Hotswap:Hotswap_Choc_V2_1.00u"
 			(at 116.84 135.89 0)
 			(hide yes)
@@
 			)
 		)
-		(property "Footprint" "ScottoKeebs_Hotswap:Hotswap_MX_1.00u"
+		(property "Footprint" "ScottoKeebs_Hotswap:Hotswap_Choc_V2_1.00u"
 			(at 91.44 40.64 0)
 			(hide yes)
@@
 			)
 		)
-		(property "Footprint" "ScottoKeebs_Hotswap:Hotswap_MX_1.00u"
+		(property "Footprint" "ScottoKeebs_Hotswap:Hotswap_Choc_V2_1.00u"
 			(at 40.64 154.94 0)
 			(hide yes)
@@
 			)
 		)
-		(property "Footprint" "ScottoKeebs_Hotswap:Hotswap_MX_1.00u"
+		(property "Footprint" "ScottoKeebs_Hotswap:Hotswap_Choc_V2_1.00u"
 			(at 66.04 97.79 0)
 			(hide yes)
@@
 			)
 		)
-		(property "Footprint" "ScottoKeebs_Hotswap:Hotswap_MX_1.00u"
+		(property "Footprint" "ScottoKeebs_Hotswap:Hotswap_Choc_V2_1.00u"
 			(at 66.04 116.84 0)
 			(hide yes)
@@
 			)
 		)
-		(property "Footprint" "ScottoKeebs_Hotswap:Hotswap_MX_1.00u"
+		(property "Footprint" "ScottoKeebs_Hotswap:Hotswap_Choc_V2_1.00u"
 			(at 53.34 78.74 0)
 			(hide yes)
@@
 			)
 		)
-		(property "Footprint" "ScottoKeebs_Hotswap:Hotswap_MX_1.00u"
+		(property "Footprint" "ScottoKeebs_Hotswap:Hotswap_Choc_V2_1.00u"
 			(at 66.04 40.64 0)
 			(hide yes)
@@
 			)
 		)
-		(property "Footprint" "ScottoKeebs_Hotswap:Hotswap_MX_1.00u"
+		(property "Footprint" "ScottoKeebs_Hotswap:Hotswap_Choc_V2_1.00u"
 			(at 78.74 40.64 0)
 			(hide yes)
@@
 			)
 		)
-		(property "Footprint" "ScottoKeebs_Hotswap:Hotswap_MX_1.00u"
+		(property "Footprint" "ScottoKeebs_Hotswap:Hotswap_Choc_V2_1.00u"
 			(at 116.84 59.69 0)
 			(hide yes)
@@
 			)
 		)
-		(property "Footprint" "ScottoKeebs_Hotswap:Hotswap_MX_1.00u"
+		(property "Footprint" "ScottoKeebs_Hotswap:Hotswap_Choc_V2_1.00u"
 			(at 104.14 116.84 0)
 			(hide yes)
@@
 			)
 		)
-		(property "Footprint" "ScottoKeebs_Hotswap:Hotswap_MX_1.00u"
+		(property "Footprint" "ScottoKeebs_Hotswap:Hotswap_Choc_V2_1.00u"
 			(at 66.04 59.69 0)
 			(hide yes)
@@
 			)
 		)
-		(property "Footprint" "ScottoKeebs_Hotswap:Hotswap_MX_1.00u"
+		(property "Footprint" "ScottoKeebs_Hotswap:Hotswap_Choc_V2_1.00u"
 			(at 78.74 135.89 0)
 			(hide yes)
@@
 			)
 		)
-		(property "Footprint" "ScottoKeebs_Hotswap:Hotswap_MX_1.00u"
+		(property "Footprint" "ScottoKeebs_Hotswap:Hotswap_Choc_V2_1.00u"
 			(at 91.44 59.69 0)
 			(hide yes)
@@
 			)
 		)
-		(property "Footprint" "ScottoKeebs_Hotswap:Hotswap_MX_1.00u"
+		(property "Footprint" "ScottoKeebs_Hotswap:Hotswap_Choc_V2_2.00u_90deg"
 			(at 129.54 86.36 0)
 			(hide yes)
@@
 			)
 		)
-		(property "Footprint" "ScottoKeebs_Hotswap:Hotswap_MX_1.00u"
+		(property "Footprint" "ScottoKeebs_Hotswap:Hotswap_Choc_V2_1.00u"
 			(at 91.44 135.89 0)
 			(hide yes)
